Commit message: Added frames to end effectors in arms

File: ros2_humanoid_virtual_twin/description/RobotElements/LeftArmElems/Lforearm.xacro (robot description, xacro)
@@ -52,3 +52,9 @@
         </xacro:if>
     </gazebo>
+    <link name="Left_End_Effector"/>
+    <joint name="LEF" type="fixed">
+        <origin xyz="0 0 -112.3e-3" rpy="0 0 0"/>
+        <parent link="Left_Forearm"/>
+        <child link="Left_End_Effector"/>
+    </joint>
 </robot>

File: ros2_humanoid_virtual_twin/description/RobotElements/RightArmElems/Rforearm.xacro (robot description, xacro)
@@ -52,3 +52,9 @@
         </xacro:if>
     </gazebo>
+    <link name="Right_End_Effector"/>
+    <joint name="REF" type="fixed">
+        <origin xyz="0 0 -112.3e-3" rpy="0 0 0"/>
+        <parent link="Right_Forearm"/>
+        <child link="Right_End_Effector"/>
+    </joint>
 </robot>

File: ros2_humanoid_virtual_twin/description/RobotElements/left_arm.xacro (robot description, xacro)
@@ -3,4 +3,4 @@
   <xacro:include filename="LeftArmElems/Larmmount.xacro"/>
   <xacro:include filename="LeftArmElems/Larm.xacro"/>
-  <!-- <xacro:include filename="LeftArmElems/Lforearm.xacro"/> -->
+  <xacro:include filename="LeftArmElems/Lforearm.xacro"/>
 </robot>

File: ros2_humanoid_virtual_twin/description/RobotElements/right_arm.xacro (robot description, xacro)
@@ -3,4 +3,4 @@
   <xacro:include filename="RightArmElems/Rarmmount.xacro"/>
   <xacro:include filename="RightArmElems/Rarm.xacro"/>
-  <!-- <xacro:include filename="RightArmElems/Rforearm.xacro"/> -->
+  <xacro:include filename="RightArmElems/Rforearm.xacro"/>
 </robot>
